File: mk_vco/mk_vco.kicad_pcb (KiCad board)
At the start: 2 copper layers, 165.3 x 128.5 mm, 67 parts, among them J1 Conn_02x05_Odd_Even, J2 1V/OCT, J3 FM CV, J4 PWM CV, J5 SAW OUT, J6 PULSE OUT, Q1 BC558, Q2 BC548, U1 TL074, U2 40106

Commit message: reorganize
Parts:
- C3, C4: footprint Capacitor_THT:CP_Radial_D8.0mm_P5.00mm -> Capacitor_THT:CP_Radial_D6.3mm_P2.50mm
Routing:
- net -12V: track 188.9 -> 186.2 mm
