File: mk_vco/mk_vco.kicad_sch (KiCad schematic)
At the start: 55 parts, among them J1 Conn_02x05_Odd_Even, J2 1V/OCT, J3 FM CV, J4 PWM CV, J5 SAW OUT, J6 PULSE OUT, Q1 BC558, Q2 BC548, U1 TL074, U2 40106

Commit message: reorganize
Parts:
- C3, C4: footprint Capacitor_THT:CP_Radial_D8.0mm_P5.00mm -> Capacitor_THT:CP_Radial_D6.3mm_P2.50mm
Connections:
- net GND: no longer J1.3 (Pin_3), J1.7 (Pin_7)
- new net: J1.3 (Pin_3), J1.7 (Pin_7)
Changed lines of the file:
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@@
 	)
 	(junction
-		(at 44.45 229.87)
-		(diameter 0)
-		(color 0 0 0 0)
-	)
-	(junction
 		(at 81.28 115.57)
 		(diameter 0)
@@
 		(at 219.71 219.71)
 	)
+	(bus_entry
+		(at 439.42 80.01)
+		(size 2.54 2.54)
+		(stroke
+			(width 0)
+			(type default)
+		)
+	)
 	(wire
 		(pts
@@
 	(wire
 		(pts
-			(xy 41.91 229.87) (xy 44.45 229.87)
+			(xy 41.91 229.87) (xy 48.26 229.87)
 		)
 		(stroke
@@
 	(wire
 		(pts
-			(xy 44.45 229.87) (xy 44.45 232.41)
-		)
-		(stroke
-			(width 0)
-			(type default)
-		)
-	)
-	(wire
-		(pts
 			(xy 26.67 229.87) (xy 29.21 229.87)
 		)
@@
 	(wire
 		(pts
-			(xy 44.45 229.87) (xy 48.26 229.87)
-		)
-		(stroke
-			(width 0)
-			(type default)
-		)
-	)
-	(wire
-		(pts
 			(xy 153.67 213.36) (xy 153.67 215.9)
 		)
@@
 	(wire
 		(pts
-			(xy 44.45 227.33) (xy 44.45 229.87)
+			(xy 44.45 227.33) (xy 44.45 232.41)
 		)
 		(stroke
@@
 			)
 		)
-		(property "Footprint" "Capacitor_THT:CP_Radial_D8.0mm_P5.00mm"
+		(property "Footprint" "Capacitor_THT:CP_Radial_D6.3mm_P2.50mm"
 			(at 64.135 229.235 0)
 			(effects
@@
 			)
 		)
-		(property "Footprint" "Capacitor_THT:CP_Radial_D8.0mm_P5.00mm"
+		(property "Footprint" "Capacitor_THT:CP_Radial_D6.3mm_P2.50mm"
 			(at 64.135 240.665 0)
 			(effects
