File: 555_eg/555_eg.kicad_pcb (KiCad board)
At the start: 2 copper layers, 168.2 x 128.5 mm, 56 parts, among them J1 Gate In, J2 Envelope Out, J3 Inverted Out, J4 Power Connector, Q1 2N3904, Q2 2N3904, Q3 2N3904, U1 NE555P, U2 TL074

Commit message: Finish eg pcb, almost done panel
Parts:
- removed ?: , 
- removed the REF** at (101.3, 132.0)
- removed the REF** at (86.1, 31.5)
- removed the REF** at (86.1, 132.0)
- removed the REF** at (101.3, 31.5)
- added REF**: MountingHole_3.2mm_M3, MountingHole:MountingHole_3.2mm_M3, F.Cu at (104.8, 48.3)
- added REF**: MountingHole_3.2mm_M3, MountingHole:MountingHole_3.2mm_M3, F.Cu at (81.8, 114.8)
- J4: moved to B.Cu
- moved REF** 96.5 mm to (204.5, 45.5)
- moved R12 90.5 mm to (105.5, 88.3), turned to -90 degrees
- moved J3 88.6 mm to (105.3, 103.4)
- moved R7 87.9 mm to (102.7, 63.7), turned to 180 degrees
- moved R2 85.9 mm to (100.1, 37.5), turned to 180 degrees
- moved J4 85.3 mm to (102.5, 117.8), turned to 180 degrees
- moved R3 84.5 mm to (99.5, 52.1), turned to 90 degrees
- moved R5 82.7 mm to (96.0, 44.4), turned to -90 degrees
- moved J1 81.9 mm to (81.5, 108.5), turned to 180 degrees
- moved J2 81.6 mm to (85.5, 108.5), turned to 180 degrees
- moved R4 80.8 mm to (94.2, 41.2), turned to 180 degrees
- moved R6 80.3 mm to (93.0, 46.5), turned to 180 degrees
- moved R11 78.6 mm to (91.5, 104.0), turned to 90 degrees
- moved D1 77.0 mm to (98.4, 30.5)
- moved R10 75.8 mm to (90.5, 88.5), turned to 90 degrees
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Connections:
- J1 pad S: Net-(J1-PadS) -> GND
- J1 pad TN: Net-(J1-PadS) -> GND
Routing:
- net +12V: track 0.00 -> 126.9 mm
- net Net-(J1-PadT): track 0.00 -> 72.8 mm
- net Net-(D3-A): track 0.00 -> 68.2 mm, vias 0 -> 1
- net -12V: track 0.00 -> 55.8 mm
- net Net-(Q2-C): track 0.00 -> 46.4 mm, vias 0 -> 1
- net Net-(Q2-B): track 0.00 -> 26.6 mm, vias 0 -> 1
- net Net-(U2B--): track 0.00 -> 26.4 mm
- net Net-(Q3-C): track 0.00 -> 26.3 mm
- net Net-(U1-DIS): track 0.00 -> 25.5 mm
- net Net-(U1-Q): track 0.00 -> 21.9 mm
- net Net-(J3-PadT): track 0.00 -> 20.6 mm
- net Net-(D1-K): track 0.00 -> 20.6 mm
- net Net-(D2-K): track 0.00 -> 18.9 mm
- net Net-(D7-K): track 0.00 -> 18.7 mm
- net Net-(U2C--): track 0.00 -> 16.5 mm
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- added copper zone on B.Cu, net GND
Other:
- board size 168.2 x 128.5 mm -> 151.7 x 128.5 mm
- board text added: "A"
- board text added: "D"
- board text added: "ENV"
- board text added: "GATE"
- board text added: "INV"
- board text added: "R"
- board text added: "S"
- board text removed: "FINE"
- board text removed: "FM"
- board text removed: "FM LEVEL"
- board text removed: "PULSE"
- board text removed: "PULSE WIDTH"
- board text removed: "PWM LEVEL"
- board text removed: "SAW"
- board text removed: "V/OCT"

Commit message: final changes to 555 EG and fixed VCA pcb before ordering
Parts:
- removed the REF** at (206.0, 36.5)
- removed the REF** at (204.5, 45.5)
- removed the REF** at (172.6, 150.5)
- removed the REF** at (157.4, 150.5)
- removed the REF** at (157.4, 28.0)
- removed the REF** at (153.5, 122.5)
- removed the REF** at (176.5, 56.0)
- removed the REF** at (172.6, 28.0)
- moved D6 58.3 mm to (150.5, 127.8)
- moved R2 58.3 mm to (156.6, 52.0)
- moved RV2 58.3 mm to (144.6, 82.5)
- moved C1 58.3 mm to (143.5, 64.5)
- moved C2 58.3 mm to (151.0, 73.5)
- moved C3 58.3 mm to (157.5, 84.5)
- moved C4 58.3 mm to (138.0, 145.5)
- moved C5 58.3 mm to (145.5, 145.5)
- moved C6 58.3 mm to (151.5, 111.0)
- moved C7 58.3 mm to (151.5, 115.0)
- moved C8 58.3 mm to (151.5, 119.1)
- moved C9 58.3 mm to (151.5, 123.5)
- moved D1 58.3 mm to (154.9, 45.0)
- moved D2 58.3 mm to (149.5, 48.5)
- moved D3 58.3 mm to (161.5, 88.4)
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Other:
- board size 151.7 x 128.5 mm -> 29 x 106.5 mm
- board text added: "555 EG Jesse Holzman"
- board text removed: "555 EG"
- board text removed: "A"
- board text removed: "COARSE"
- board text removed: "D"
- board text removed: "ENV"
- board text removed: "GATE"
- board text removed: "INV"
- board text removed: "PWM"
- board text removed: "R"
- board text removed: "S"
