File: 555_eg/555_eg_PANEL.kicad_pcb (KiCad board)
At the start: 2 copper layers, 30 x 128.5 mm, 6 parts

Commit message: final changes to 555 EG and fixed VCA pcb before ordering
Other:
- outline, holes or cut-outs redrawn
- board text added: "RELEASE"
- board text added: "SUSTAIN"
- board text removed: "R"
- board text removed: "S"
