File: 555_eg/555_eg.kicad_sch (KiCad schematic)
At the start: 43 parts, among them J1 Gate In, J2 Envelope Out, J3 Inverted Out, J4 Power Connector, Q1 2N3904, Q2 2N3904, Q3 2N3904, U1 NE555P, U2 TL074

Commit message: Swap out pot and resistor values for better ADSR values, fix sustain pot pins
Parts:
- R10, R7, R8: value 100k -> 220
- RV1, RV2, RV4: value A1M -> A100k
Connections:
- net at R9.1: now also RV3.3; no longer RV3.1
- net at U1.7 (DIS): now also RV3.1; no longer RV3.3
Changed lines of the file:
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@@
 			)
 		)
-		(property "Value" "100k"
+		(property "Value" "220"
 			(at 186.69 40.64 90)
 			(effects
@@
 			)
 		)
-		(property "Value" "A1M"
+		(property "Value" "A100k"
 			(at 194.31 74.9299 0)
 			(effects
@@
 			)
 		)
-		(property "Value" "A1M"
+		(property "Value" "A100k"
 			(at 218.44 105.4099 0)
 			(effects
@@
 			)
 		)
-		(property "Value" "100k"
+		(property "Value" "220"
 			(at 186.69 64.77 90)
 			(effects
@@
 		(lib_id "Device:R_Potentiometer_US")
 		(at 198.12 121.92 0)
+		(mirror x)
 		(unit 1)
 		(exclude_from_sim no)
@@
 		(dnp no)
 		(property "Reference" "RV3"
-			(at 195.58 120.6499 0)
+			(at 195.58 123.1901 0)
 			(effects
 				(font
@@
 		)
 		(property "Value" "B10K"
-			(at 195.58 123.1899 0)
+			(at 195.58 120.6501 0)
 			(effects
 				(font
@@
 		)
 		(property "Label" "Sustain"
-			(at 191.516 125.476 0)
+			(at 191.516 118.364 0)
 			(effects
 				(font
@@
 			)
 		)
-		(property "Value" "A1M"
+		(property "Value" "A100k"
 			(at 194.31 50.7999 0)
 			(effects
@@
 			)
 		)
-		(property "Value" "100k"
+		(property "Value" "220"
 			(at 223.52 118.1099 0)
 			(effects
