File: mix4/mix4.kicad_pcb (KiCad board)
At the start: 2 copper layers, 29 x 106.5 mm, 31 parts, among them J1 Input A, J2 Input B, J3 Input C, J4 Input D, J5 Mix Out, J6 Power Connector, U1 TL074

Commit message: progress on mixer pcb
Parts:
- removed the REF** at (125.0, 146.5)
- removed the REF** at (109.8, 46.0)
- added REF**: MountingHole_3.2mm_M3, MountingHole:MountingHole_3.2mm_M3, F.Cu at (176.0, 157.0)
- added REF**: MountingHole_3.2mm_M3, MountingHole:MountingHole_3.2mm_M3, F.Cu at (201.4, 157.0)
- added REF**: MountingHole_3.2mm_M3, MountingHole:MountingHole_3.2mm_M3, F.Cu at (176.0, 34.5)
- added REF**: MountingHole_3.2mm_M3, MountingHole:MountingHole_3.2mm_M3, F.Cu at (201.4, 34.5)
- J1, J2, J3, J4, J5: footprint Library:PinHeader_1x03_P2.54mm_Vertical_AudioJack -> Connector_Audio:Jack_3.5mm_QingPu_WQP-PJ398SM_Vertical_CircularHoles
- RV1, RV2, RV3, RV4, RV5: footprint Connector_PinHeader_2.54mm:PinHeader_1x03_P2.54mm_Vertical -> Potentiometer_THT:Potentiometer_Alpha_RD901F-40-00D_Single_Vertical_CircularHoles
- moved J5 145.2 mm to (247.2, 134.0)
- moved J4 126.0 mm to (230.2, 111.5)
- moved RV4 124.5 mm to (244.7, 125.5), turned to 90 degrees
- moved J3 124.2 mm to (230.2, 89.0)
- moved J1 124.0 mm to (230.2, 44.0)
- moved J2 123.7 mm to (230.2, 66.5)
- moved RV3 120.6 mm to (244.7, 103.0), turned to 90 degrees
- moved RV2 117.8 mm to (244.7, 80.5), turned to 90 degrees
- moved RV1 116.2 mm to (244.7, 58.0), turned to 90 degrees
- moved RV5 114.5 mm to (227.7, 148.0), turned to 90 degrees
- moved J6 56.1 mm to (71.5, 121.8)
- moved R1 39.6 mm to (85.5, 38.9)
- moved R2 23.3 mm to (76.3, 82.7)
- moved R3 23.3 mm to (76.3, 86.8)
- moved R4 23.3 mm to (76.3, 90.8)
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Other:
- board size 29 x 106.5 mm -> 89.8 x 128.5 mm
- board text added: "A"
- board text added: "COARSE"
- board text added: "MIXER"
- board text added: "OUT"

Commit message: mixer pcb almost done :)
Parts:
- added J10: ~, Connector_PinHeader_2.54mm:PinHeader_1x03_P2.54mm_Vertical, B.Cu at (108.0, 136.0)
- added J11: Conn_01x03, Connector_PinSocket_2.54mm:PinSocket_1x03_P2.54mm_Vertical, F.Cu at (148.0, 136.0)
- added J6: Conn_01x03, Connector_PinHeader_2.54mm:PinHeader_1x03_P2.54mm_Vertical, B.Cu at (132.9, 65.0)
- added J7: ~, Connector_PinSocket_2.54mm:PinSocket_1x03_P2.54mm_Vertical, F.Cu at (172.9, 65.0)
- added J8: Conn_01x03, Connector_PinHeader_2.54mm:PinHeader_1x03_P2.54mm_Vertical, B.Cu at (132.9, 110.0)
- added J9: ~, Connector_PinSocket_2.54mm:PinSocket_1x03_P2.54mm_Vertical, F.Cu at (172.9, 110.0)
- moved REF** 123.9 mm to (77.5, 161.0)
- moved REF** 123.9 mm to (77.5, 38.5)
- moved RV1 121.5 mm to (123.2, 62.0)
- moved RV2 121.5 mm to (123.2, 84.5)
- moved RV3 121.5 mm to (123.2, 107.0)
- moved RV4 121.5 mm to (123.2, 129.5)
- moved J1 118.8 mm to (111.4, 48.0)
- moved J2 118.8 mm to (111.4, 70.5)
- moved J3 118.8 mm to (111.4, 93.0)
- moved J4 118.8 mm to (111.4, 115.5)
- moved J5 117.8 mm to (129.4, 138.0)
- moved RV5 115.1 mm to (112.6, 152.0)
- moved REF** 113.8 mm to (62.3, 161.0)
- moved REF** 113.8 mm to (62.3, 38.5)
- moved J12 99.4 mm to (170.9, 122.8)
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- renumbered J6 to J12
Connections:
- net Net-(J5-PadT) renamed MIX_OUT
- net Net-(R1-Pad1) renamed INPUT_A
- net Net-(R2-Pad1) renamed INPUT_B
- net Net-(R3-Pad1) renamed INPUT_C
- net Net-(R4-Pad1) renamed INPUT_D
- net Net-(R5-Pad1) renamed MIX_GAIN_2
- net Net-(U1A--) renamed MIX_GAIN_1
Routing:
- net MIX_GAIN_1: track 0.00 -> 128.2 mm, vias 0 -> 1
- net MIX_GAIN_2: track 0.00 -> 97.7 mm
- net MIX_OUT: track 0.00 -> 82.9 mm, vias 0 -> 1
- net +12V: track 0.00 -> 78.7 mm, vias 0 -> 1
- net INPUT_D: track 0.00 -> 65.0 mm
- net INPUT_C: track 0.00 -> 61.5 mm, vias 0 -> 1
- net -12V: track 0.00 -> 57.5 mm, vias 0 -> 1
- net INPUT_B: track 0.00 -> 42.8 mm
- net INPUT_A: track 0.00 -> 34.0 mm
- net Net-(R6-Pad2): track 0.00 -> 22.8 mm
- net Net-(J4-PadT): track 0.00 -> 19.5 mm
- net Net-(J2-PadT): track 0.00 -> 19.5 mm
- net Net-(J1-PadT): track 0.00 -> 17.9 mm
- net Net-(J3-PadT): track 0.00 -> 17.9 mm
- net Net-(U1B--): track 0.00 -> 16.2 mm
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- added copper zone on B.Cu, net GND
Other:
- board size 89.8 x 128.5 mm -> 120 x 128.5 mm
- board text added: "B"
- board text added: "C"
- board text added: "D"
- board text added: "MIX LEVEL"
- board text removed: "COARSE"
