File: mix4/mix4.kicad_pcb (KiCad board)
At the start: 2 copper layers, 120 x 128.5 mm, 39 parts, among them J1 Input A, J11 Conn_01x03, J12 Power Connector, J2 Input B, J3 Input C, J4 Input D, J5 Mix Out, J6 Conn_01x03, J8 Conn_01x03, U1 TL074

Commit message: split main board and control board grounds in mixer pcb
Connections:
- J1 pad S: GND -> CTRL_GND
- J1 pad TN: GND -> CTRL_GND
- J10 pad 1: MIX_GAIN_1 -> MIX_GAIN_1_CTRL
- J10 pad 2: MIX_GAIN_2 -> MIX_GAIN_2_CTRL
- J10 pad 3: MIX_OUT -> MIX_OUT_CTRL
- J2 pad S: GND -> CTRL_GND
- J2 pad TN: GND -> CTRL_GND
- J3 pad S: GND -> CTRL_GND
- J3 pad TN: GND -> CTRL_GND
- J4 pad S: GND -> CTRL_GND
- J4 pad TN: GND -> CTRL_GND
- J5 pad S: GND -> CTRL_GND
- J5 pad T: MIX_OUT -> MIX_OUT_CTRL
- J5 pad TN: GND -> CTRL_GND
- J6 pad 1: INPUT_A -> INPUT_A_CTRL
- J6 pad 2: INPUT_B -> INPUT_B_CTRL
- J6 pad 3: GND -> CTRL_GND
- J8 pad 1: INPUT_C -> INPUT_C_CTRL
- J8 pad 2: INPUT_D -> INPUT_D_CTRL
- J8 pad 3: GND -> CTRL_GND
- RV1 pad 1: GND -> CTRL_GND
- RV1 pad 2: INPUT_A -> INPUT_A_CTRL
- RV2 pad 1: GND -> CTRL_GND
- RV2 pad 2: INPUT_B -> INPUT_B_CTRL
- RV3 pad 1: GND -> CTRL_GND
- RV3 pad 2: INPUT_C -> INPUT_C_CTRL
- RV4 pad 1: GND -> CTRL_GND
- RV4 pad 2: INPUT_D -> INPUT_D_CTRL
- RV5 pad 1: MIX_GAIN_1 -> MIX_GAIN_1_CTRL
- RV5 pad 2: MIX_GAIN_2 -> MIX_GAIN_2_CTRL
- RV5 pad 3: MIX_GAIN_2 -> MIX_GAIN_2_CTRL
Routing:
- net MIX_OUT_CTRL: track 0.00 -> 29.0 mm
- net MIX_OUT: track 82.9 -> 53.9 mm
- net MIX_GAIN_2: track 97.7 -> 73.7 mm
- net MIX_GAIN_2_CTRL: track 0.00 -> 24.0 mm
- net INPUT_D: track 65.0 -> 42.4 mm
- net INPUT_D_CTRL: track 0.00 -> 22.5 mm
- net INPUT_B_CTRL: track 0.00 -> 22.2 mm
- net INPUT_B: track 42.8 -> 20.6 mm
- net MIX_GAIN_1_CTRL: track 0.00 -> 17.9 mm
- net MIX_GAIN_1: track 128.2 -> 110.3 mm
- net INPUT_A_CTRL: track 0.00 -> 8.45 mm
- net INPUT_A: track 34.0 -> 25.5 mm
- net INPUT_C: track 61.5 -> 53.0 mm
- net INPUT_C_CTRL: track 0.00 -> 8.43 mm
- added copper zone on B.Cu, net CTRL_GND

Commit message: Add title+revision labels to mixer boards
Other:
- board text added: "4-Channel Mixer [Rev 1] Control Board Jesse Holzman 2026"
- board text added: "4-Channel Mixer [Rev 1] Main Board Jesse Holzman 2026"
