File: mix4/mix4.kicad_sch (KiCad schematic)
At the start: 29 parts, among them J1 Input A, J2 Input B, J3 Input C, J4 Input D, J5 Mix Out, J6 Power Connector, U1 TL074

Commit message: mixer pcb almost done :)
Parts:
- added J10: ~, Connector_PinHeader_2.54mm:PinHeader_1x03_P2.54mm_Vertical, symbol Connector_Generic:Conn_01x03
- added J11: Conn_01x03, Connector_PinSocket_2.54mm:PinSocket_1x03_P2.54mm_Vertical, symbol Connector_Generic:Conn_01x03
- added J6, J8: Conn_01x03, Connector_PinHeader_2.54mm:PinHeader_1x03_P2.54mm_Vertical, symbol Connector_Generic:Conn_01x03
- added J7, J9: ~, Connector_PinSocket_2.54mm:PinSocket_1x03_P2.54mm_Vertical, symbol Connector_Generic:Conn_01x03
- J1, J2, J3, J4, J5: footprint Library:PinHeader_1x03_P2.54mm_Vertical_AudioJack -> Connector_Audio:Jack_3.5mm_QingPu_WQP-PJ398SM_Vertical_CircularHoles
- RV1, RV2, RV3, RV4, RV5: footprint Connector_PinHeader_2.54mm:PinHeader_1x03_P2.54mm_Vertical -> Potentiometer_THT:Potentiometer_Alpha_RD901F-40-00D_Single_Vertical_CircularHoles
- renumbered J6 to J12
Connections:
- net GND: now also J6.3 (Pin_3), J7.3 (Pin_3), J8.3 (Pin_3), J9.3 (Pin_3)
- net INPUT_D: now reaches R4.1, RV4.2
- net INPUT_D: now also J8.2 (Pin_2), J9.2 (Pin_2)
- net INPUT_A: now reaches R1.1, RV1.2
- net INPUT_A: now also J6.1 (Pin_1), J7.1 (Pin_1)
- net MIX_GAIN_2: now reaches R5.1, RV5.2, RV5.3, U1.1
- net MIX_GAIN_2: now also J10.2 (Pin_2), J11.2 (Pin_2)
- net MIX_GAIN_1: now reaches R1.2, R2.2, R3.2, R4.2, RV5.1, U1.2 (-)
- net MIX_GAIN_1: now also J10.1 (Pin_1), J11.1 (Pin_1)
- net MIX_OUT: now reaches J5.T, R7.2
- net MIX_OUT: now also J10.3 (Pin_3), J11.3 (Pin_3)
- net INPUT_C: now reaches R3.1, RV3.2
- net INPUT_C: now also J8.1 (Pin_1), J9.1 (Pin_1)
- net INPUT_B: now reaches R2.1, RV2.2
- net INPUT_B: now also J6.2 (Pin_2), J7.2 (Pin_2)
Other:
- moved on the sheet: J1, J2, J3, J4, J5, R1, R2, R3, R4, R5, R6, R7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

Commit message: split main board and control board grounds in mixer pcb
Connections:
- net GND: no longer J1.S, J1.TN, J2.S, J2.TN, J3.S, J3.TN, J4.S, J4.TN, J5.S, J5.TN, J6.3 (Pin_3), J8.3 (Pin_3), RV1.1, RV2.1, RV3.1, RV4.1
- net INPUT_A: no longer J6.1 (Pin_1), RV1.2
- net INPUT_B: no longer J6.2 (Pin_2), RV2.2
- net INPUT_C: no longer J8.1 (Pin_1), RV3.2
- net INPUT_D: no longer J8.2 (Pin_2), RV4.2
- net MIX_GAIN_1: no longer J10.1 (Pin_1), RV5.1
- net MIX_GAIN_2: no longer J10.2 (Pin_2), RV5.2, RV5.3
- net MIX_OUT: no longer J10.3 (Pin_3), J5.T
- new net CTRL_GND: J1.S, J1.TN, J2.S, J2.TN, J3.S, J3.TN, J4.S, J4.TN, J5.S, J5.TN, J6.3 (Pin_3), J8.3 (Pin_3), RV1.1, RV2.1, RV3.1, RV4.1
- new net INPUT_A_CTRL: J6.1 (Pin_1), RV1.2
- new net INPUT_B_CTRL: J6.2 (Pin_2), RV2.2
- new net INPUT_C_CTRL: J8.1 (Pin_1), RV3.2
- new net INPUT_D_CTRL: J8.2 (Pin_2), RV4.2
- new net MIX_GAIN_1_CTRL: J10.1 (Pin_1), RV5.1
- new net MIX_GAIN_2_CTRL: J10.2 (Pin_2), RV5.2, RV5.3
- new net MIX_OUT_CTRL: J10.3 (Pin_3), J5.T
