File: simple_lfo/simple_lfo.kicad_sch (KiCad schematic)
At the start: 40 parts, among them J1 LFO Out, J10 To J3, J11 To J4 (Range Switch), J12 To J3, J2 Power Connector, J3 To J4 (Range Switch), J4 To J3, J5 Conn_01x03_Pin, J6 To J3, J7 To J4 (Range Switch), J8 To J3, J9 To J4 (Range Switch), SW1 Range, SW2 Waveform, U1 TL074

Commit message: LFO: All components on pcbs laid out
Parts:
- J1: renamed from J6; footprint (none) -> Connector_PinSocket_2.54mm:PinSocket_1x03_P2.54mm_Vertical
- J10: renamed from J11; footprint (none) -> Connector_PinHeader_2.54mm:PinHeader_1x03_P2.54mm_Vertical
- J11: renamed from J12; footprint (none) -> Connector_PinSocket_2.54mm:PinSocket_1x03_P2.54mm_Vertical
- J2: renamed from J5; footprint (none) -> Connector_PinHeader_2.54mm:PinHeader_1x03_P2.54mm_Vertical
- J3: footprint (none) -> Connector_PinHeader_2.54mm:PinHeader_1x03_P2.54mm_Vertical
- J4: footprint (none) -> Connector_PinSocket_2.54mm:PinSocket_1x03_P2.54mm_Vertical
- J5: renamed from J7; footprint (none) -> Connector_PinHeader_2.54mm:PinHeader_1x03_P2.54mm_Vertical
- J6: renamed from J8; footprint (none) -> Connector_PinSocket_2.54mm:PinSocket_1x03_P2.54mm_Vertical
- J7: renamed from J9; footprint (none) -> Connector_PinHeader_2.54mm:PinHeader_1x03_P2.54mm_Vertical
- J8: renamed from J10; footprint (none) -> Connector_PinSocket_2.54mm:PinSocket_1x03_P2.54mm_Vertical
- renumbered J2 to J12, J1 to J9
Connections:
- net GND: now also J10.3 (Pin_3); no longer RV2.1
- net CTRL_PANEL_GND: now reaches J11.3 (Pin_3)
- net CTRL_PANEL_GND: now also J8.1 (Pin_1), J8.3 (Pin_3), J9.S, J9.TN, RV2.1
- no-connect marks 2 -> 0
Other:
- moved on the sheet: C1, C2, D1, J1, J10, J11, J2, J3, J4, J5, J6, J7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
