File: 2164_vca/2164_vca.kicad_sch (KiCad schematic)
At the start: 14 parts, among them J1 Power Connector, U1 SSI2164, U2 TL074

Commit message: 2164 vca: assigned missing footprints and some tweaks
Parts:
- D1: footprint (none) -> Diode_THT:D_DO-41_SOD81_P10.16mm_Horizontal
Connections:
- net -12V: no longer D1.2 (A)
- net VCA_A/VCA1_CV renamed VCA1_CV
- net VCA_A/VCA1_IN renamed VCA1_IN
- net VCA_A/VCA1_OUT renamed VCA1_OUT
- net VCA_A/VCA2_CV renamed VCA2_CV
- net VCA_A/VCA2_IN renamed VCA2_IN
- net VCA_A/VCA2_OUT renamed VCA2_OUT
- net VCA_B/VCA3_CV renamed VCA3_CV
- net VCA_B/VCA3_IN renamed VCA3_IN
- net VCA_B/VCA3_OUT renamed VCA3_OUT
- net VCA_B/VCA4_CV renamed VCA4_CV
- net VCA_B/VCA4_IN renamed VCA4_IN
- net VCA_B/VCA4_OUT renamed VCA4_OUT
Other:
- sheet VCA_A ports: added none; removed VCA1_CV, VCA1_IN, VCA1_OUT, VCA2_CV, VCA2_IN, VCA2_OUT
- sheet VCA_B ports: added none; removed VCA3_CV, VCA3_IN, VCA3_OUT, VCA4_CV, VCA4_IN, VCA4_OUT

Commit message: 2164 vca: finalized panel and control board layout
Connections:
- net -12V: now also D1.2 (A)
Changed lines of the file:
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@@
+	)
+	(junction
+		(at 72.39 116.84)
+		(diameter 0)
+		(color 0 0 0 0)
 	)
 	(junction
@@
 	(wire
 		(pts
-			(xy 72.39 113.03) (xy 72.39 119.38)
+			(xy 72.39 113.03) (xy 72.39 116.84)
 		)
 		(stroke
@@
 	(wire
 		(pts
+			(xy 72.39 116.84) (xy 72.39 119.38)
+		)
+		(stroke
+			(width 0)
+			(type default)
+		)
+	)
+	(wire
+		(pts
 			(xy 138.43 127) (xy 144.78 127)
 		)
@@
 		)
 		(stroke
+			(width 0)
+			(type default)
+		)
+	)
+	(wire
+		(pts
+			(xy 72.39 116.84) (xy 78.74 116.84)
+		)
+		(stroke
