File: 2164_vca/vca_a.kicad_sch (KiCad schematic)
At the start: 27 parts, among them J10 Conn_01x03_Pin, J2 CV A, J3 To J3, J4 Conn_01x03_Pin, J5 To J3, J6 Conn_01x03_Pin, J7 In A, J8 Out A, J9 To J3, U2 TL074

Commit message: 2164 vca: assigned missing footprints and some tweaks
Parts:
- RV3: footprint (none) -> Potentiometer_THT:Potentiometer_Runtron_RM-065_Vertical
- RV4: value B10K -> B50K; footprint (none) -> Potentiometer_THT:Potentiometer_Runtron_RM-065_Vertical
Changed lines of the file:
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@@
+		)
+	)
+	(global_label "VCA2_CV"
+		(shape input)
+		(at 175.26 109.22 270)
+		(fields_autoplaced yes)
+		(effects
+			(font
+				(size 1.27 1.27)
+			)
+			(justify right)
+		)
+		(property "Intersheetrefs" "${INTERSHEET_REFS}"
+			(at 175.26 120.1881 90)
+			(effects
+				(font
+					(size 1.27 1.27)
+				)
+				(justify right)
+				(hide yes)
+			)
+		)
+	)
+	(global_label "VCA2_IN"
+		(shape input)
+		(at 162.56 123.19 0)
+		(fields_autoplaced yes)
+		(effects
+			(font
+				(size 1.27 1.27)
+			)
+			(justify left)
+		)
+		(property "Intersheetrefs" "${INTERSHEET_REFS}"
+			(at 173.1048 123.19 0)
+			(effects
+				(font
+					(size 1.27 1.27)
+				)
+				(justify left)
+				(hide yes)
+			)
+		)
+	)
+	(global_label "VCA1_IN"
+		(shape input)
+		(at 83.82 146.05 0)
+		(fields_autoplaced yes)
+		(effects
+			(font
+				(size 1.27 1.27)
+			)
+			(justify left)
+		)
+		(property "Intersheetrefs" "${INTERSHEET_REFS}"
+			(at 94.3648 146.05 0)
+			(effects
+				(font
+					(size 1.27 1.27)
+				)
+				(justify left)
+				(hide yes)
+			)
 		)
 	)
@@
 		)
 	)
+	(global_label "VCA1_CV"
+		(shape input)
+		(at 96.52 160.02 90)
+		(fields_autoplaced yes)
+		(effects
+			(font
+				(size 1.27 1.27)
+			)
+			(justify left)
+		)
+		(property "Intersheetrefs" "${INTERSHEET_REFS}"
+			(at 96.52 149.0519 90)
+			(effects
+				(font
+					(size 1.27 1.27)
+				)
+				(justify left)
+				(hide yes)
+			)
+		)
+	)
 	(global_label "CTRL_GND"
 		(shape passive)
@@
 		)
 	)
-	(hierarchical_label "VCA1_CV"
+	(global_label "VCA1_OUT"
 		(shape input)
-		(at 96.52 160.02 90)
+		(at 110.49 146.05 180)
+		(fields_autoplaced yes)
 		(effects
 			(font
 				(size 1.27 1.27)
 			)
-			(justify left)
-		)
-	)
-	(hierarchical_label "VCA2_OUT"
+			(justify right)
+		)
+		(property "Intersheetrefs" "${INTERSHEET_REFS}"
+			(at 98.2519 146.05 0)
+			(effects
+				(font
+					(size 1.27 1.27)
+				)
+				(justify right)
+				(hide yes)
+			)
+		)
+	)
+	(global_label "VCA2_OUT"
 		(shape input)
 		(at 189.23 123.19 180)
+		(fields_autoplaced yes)
 		(effects
 			(font
@@
 			(justify right)
 		)
-	)
-	(hierarchical_label "VCA2_CV"
-		(shape input)
-		(at 175.26 109.22 270)
-		(effects
-			(font
-				(size 1.27 1.27)
-			)
-			(justify right)
-		)
-	)
-	(hierarchical_label "VCA1_OUT"
-		(shape input)
-		(at 110.49 146.05 180)
-		(effects
-			(font
-				(size 1.27 1.27)
-			)
-			(justify right)
-		)
-	)
-	(hierarchical_label "VCA2_IN"
-		(shape input)
-		(at 162.56 123.19 0)
-		(effects
-			(font
-				(size 1.27 1.27)
-			)
-			(justify left)
-		)
-	)
-	(hierarchical_label "VCA1_IN"
-		(shape input)
-		(at 83.82 146.05 0)
-		(effects
-			(font
-				(size 1.27 1.27)
-			)
-			(justify left)
+		(property "Intersheetrefs" "${INTERSHEET_REFS}"
+			(at 176.9919 123.19 0)
+			(effects
+				(font
+					(size 1.27 1.27)
+				)
+				(justify right)
+				(hide yes)
+			)
 		)
 	)
@@
 			)
 		)
-		(property "Footprint" ""
+		(property "Footprint" "Potentiometer_THT:Potentiometer_Runtron_RM-065_Vertical"
 			(at 63.5 115.57 0)
 			(effects
@@
 			)
 		)
-		(property "Value" "B10K"
+		(property "Value" "B50K"
 			(at 60.96 147.3199 0)
 			(effects
@@
 			)
 		)
-		(property "Footprint" ""
+		(property "Footprint" "Potentiometer_THT:Potentiometer_Runtron_RM-065_Vertical"
 			(at 63.5 146.05 0)
 			(effects

Commit message: 2164 vca: finalized panel and control board layout
Connections:
- net VCA1_CV: now also J6.2 (Pin_2); no longer J5.2 (Pin_2)
- net VCA2_CV: now also J6.1 (Pin_1); no longer J5.1 (Pin_1)
- net at RV5.3: now also J5.1 (Pin_1); no longer J6.1 (Pin_1)
- net at RV5.2: now also J5.2 (Pin_2); no longer J6.2 (Pin_2)
- net at J6.3 (Pin_3): now also R7.1; no longer RV5.1
- net at J5.3 (Pin_3): now also RV5.1; no longer R7.1
Other:
- moved on the sheet: J5, J6
Changed lines of the file:
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@@
 	(symbol
 		(lib_id "Connector:Conn_01x03_Pin")
-		(at 148.59 81.28 0)
+		(at 143.51 81.28 0)
+		(mirror y)
 		(unit 1)
 		(exclude_from_sim no)
@@
 		(dnp no)
 		(property "Reference" "J6"
-			(at 149.352 74.93 0)
+			(at 142.748 74.93 0)
 			(effects
 				(font
@@
 		)
 		(property "Value" "Conn_01x03_Pin"
-			(at 149.225 76.2 0)
+			(at 142.875 76.2 0)
 			(effects
 				(font
@@
 		)
 		(property "Footprint" "Connector_PinHeader_2.54mm:PinHeader_1x03_P2.54mm_Vertical"
-			(at 148.59 81.28 0)
-			(effects
-				(font
-					(size 1.27 1.27)
-				)
-				(hide yes)
-			)
-		)
-		(property "Datasheet" "~"
-			(at 148.59 81.28 0)
+			(at 143.51 81.28 0)
+			(effects
+				(font
+					(size 1.27 1.27)
+				)
+				(hide yes)
+			)
+		)
+		(property "Datasheet" "~"
+			(at 143.51 81.28 0)
 			(effects
 				(font
@@
 		)
 		(property "Description" "Generic connector, single row, 01x03, script generated"
-			(at 148.59 81.28 0)
+			(at 143.51 81.28 0)
 			(effects
 				(font
@@
 	(symbol
 		(lib_id "Connector:Conn_01x03_Socket")
-		(at 143.51 81.28 0)
+		(at 148.59 81.28 0)
+		(mirror y)
 		(unit 1)
 		(exclude_from_sim no)
@@
 		(dnp no)
 		(property "Reference" "J5"
-			(at 141.732 74.93 0)
+			(at 150.368 74.93 0)
 			(effects
 				(font
@@
 		)
 		(property "Value" "To J3"
-			(at 144.78 82.5499 0)
+			(at 147.32 82.5499 0)
 			(effects
 				(font
@@
 		)
 		(property "Footprint" "Connector_PinSocket_2.54mm:PinSocket_1x03_P2.54mm_Vertical"
-			(at 143.51 81.28 0)
-			(effects
-				(font
-					(size 1.27 1.27)
-				)
-				(hide yes)
-			)
-		)
-		(property "Datasheet" "~"
-			(at 143.51 81.28 0)
+			(at 148.59 81.28 0)
+			(effects
+				(font
+					(size 1.27 1.27)
+				)
+				(hide yes)
+			)
+		)
+		(property "Datasheet" "~"
+			(at 148.59 81.28 0)
 			(effects
 				(font
@@
 		)
 		(property "Description" "Generic connector, single row, 01x03, script generated"
-			(at 143.51 81.28 0)
-			(effects
-				(font
+			(at 148.59 81.28 0)
+			(effects
+				(font
