File: ms20_vcf/ms20_vcf.kicad_sch (KiCad schematic)
At the start: 17 parts, among them J12 Power Connector, J2 Freq CV

Commit message: ms20 vcf: add freq input section of schematic
Parts:
- added C1: 4n7, symbol Device:C
- added Q1, Q2: BC557, Package_TO_SOT_THT:TO-92_Inline, symbol Transistor_BJT:BC557
- added R4: 1K5, Resistor_THT:R_Axial_DIN0207_L6.3mm_D2.5mm_P10.16mm_Horizontal, symbol Device:R
- added R5: 470K, Resistor_THT:R_Axial_DIN0207_L6.3mm_D2.5mm_P10.16mm_Horizontal, symbol Device:R
- added R6: 4K7, Resistor_THT:R_Axial_DIN0207_L6.3mm_D2.5mm_P10.16mm_Horizontal, symbol Device:R
- added RV2: 500, symbol Device:R_Potentiometer_Trim
- added U1: TL074, Package_DIP:DIP-14_W7.62mm_Socket, symbol Amplifier_Operational:TL074
Connections:
- net +12V: now also U1.4 (V+)
- net -12V: now also R5.2, U1.11 (V-)
- net GND: now also Q2.2 (B), R4.2, U1.3 (+)
- net at R1.2, R2.2, R3.2: now also Q1.2 (B), RV2.3
- new net: R4.1, RV2.1, RV2.2
- new net: C1.1, Q1.1 (C), R5.1, U1.2 (-)
- new net: Q1.3 (E), Q2.3 (E), R6.1
- new net: C1.2, R6.2, U1.1
